Commit message: Update minerva_actuators.xacro

File: minerva/minerva_description/urdf/minerva_actuators.xacro (robot description, xacro)
@@ -21,7 +21,8 @@
   <!-- Thruster joint and link snippet -->
   <xacro:macro name="thruster_macro"
-    params="namespace thruster_id *origin">
+    params="namespace parent_link thruster_id *origin">
     <xacro:thruster_module_first_order_basic_fcn_macro
       namespace="${namespace}"
+      parent_link="${parent_link}"
       thruster_id="${thruster_id}"
       mesh_filename="${prop_mesh_file}"
@@ -31,59 +32,118 @@
     </xacro:thruster_module_first_order_basic_fcn_macro>
   </xacro:macro>
-   <xacro:thruster_macro namespace="${namespace}" thruster_id="0">
-    <origin xyz="${3*length/2} 0 ${radius*2}" rpy="${0*d2r} ${-90*d2r} ${0*d2r}"/>
+<!-- Torpedo-Shape
+  <xacro:thruster_macro namespace="${namespace}" parent_link="base_link" thruster_id="0">
+    <origin xyz="${length_1 + length_joint + 0.470} 0 ${2*radius}" rpy="${0*d2r} ${0*d2r} ${-90*d2r}"/>
   </xacro:thruster_macro>
-  <xacro:thruster_macro namespace="${namespace}" thruster_id="1">
-    <origin xyz="${3*length/2} 0 0" rpy="${0*d2r} ${90*d2r} ${0*d2r}"/>
+  <xacro:thruster_macro namespace="${namespace}" parent_link="base_link" thruster_id="1">
+    <origin xyz="${length_1 + length_joint + 0.470} 0 0" rpy="${0*d2r} ${0*d2r} ${90*d2r}"/>
   </xacro:thruster_macro>
-  <xacro:thruster_macro namespace="${namespace}" thruster_id="2">
-    <origin xyz="${3*length/2} ${radius} ${radius}" rpy="${0*d2r} ${0*d2r} ${90*d2r}"/>
+  <xacro:thruster_macro namespace="${namespace}" parent_link="base_link" thruster_id="2">
+    <origin xyz="${length_1 + length_joint + 0.370} ${radius+0.08} ${radius}" rpy="${0*d2r} ${45*d2r} ${0*d2r}"/>
   </xacro:thruster_macro>
-  <xacro:thruster_macro namespace="${namespace}" thruster_id="3">
-    <origin xyz="${3*length/2} ${-radius} ${radius}" rpy="${0*d2r} ${0*d2r} ${-90*d2r}"/>
+  <xacro:thruster_macro namespace="${namespace}" parent_link="base_link" thruster_id="3">
+    <origin xyz="${length_1 + length_joint + 0.370} ${-radius-0.08} ${radius}" rpy="${0*d2r} ${-45*d2r} ${0*d2r}"/>
   </xacro:thruster_macro>
-  <xacro:thruster_macro namespace="${namespace}" thruster_id="4">
-    <origin xyz="${7*length/2} 0 ${radius*2}" rpy="${0*d2r} ${-90*d2r} ${0*d2r}"/>
+  <xacro:thruster_macro namespace="${namespace}" parent_link="base_link" thruster_id="4">
+    <origin xyz="${length_1 + length_2 + 2*length_joint + 0.670} 0 ${2*radius}" rpy="${0*d2r} ${0*d2r} ${-90*d2r}"/>
   </xacro:thruster_macro>
-  <xacro:thruster_macro namespace="${namespace}" thruster_id="5">
-    <origin xyz="${7*length/2} 0 0" rpy="${0*d2r} ${90*d2r} ${0*d2r}"/>
+  <xacro:thruster_macro namespace="${namespace}" parent_link="base_link" thruster_id="5">
+    <origin xyz="${length_1 + length_2 + 2*length_joint + 0.670} 0 0" rpy="${0*d2r} ${0*d2r} ${90*d2r}"/>
   </xacro:thruster_macro>
-  <xacro:thruster_macro namespace="${namespace}" thruster_id="6">
-    <origin xyz="${7*length/2} ${radius} ${radius}" rpy="${0*d2r} ${0*d2r} ${90*d2r}"/>
+  <xacro:thruster_macro namespace="${namespace}" parent_link="base_link" thruster_id="6">
+    <origin xyz="${length_1 + length_2 + 2*length_joint + 0.770} ${radius+0.08} ${radius}" rpy="${0*d2r} ${45*d2r} ${0*d2r}"/>
   </xacro:thruster_macro>
-  <xacro:thruster_macro namespace="${namespace}" thruster_id="7">
-    <origin xyz="${7*length/2} ${-radius} ${radius}" rpy="${0*d2r} ${0*d2r} ${-90*d2r}"/>
+  <xacro:thruster_macro namespace="${namespace}" parent_link="base_link" thruster_id="7">
+    <origin xyz="${length_1 + length_2 + 2*length_joint + 0.770} ${-radius-0.08} ${radius}" rpy="${0*d2r} ${-45*d2r} ${0*d2r}"/>
   </xacro:thruster_macro>
-  <!--
-   <xacro:thruster_macro namespace="${namespace}" thruster_id="0">
-   rotor_constant="0.00031">
-    <origin xyz="0.48 0.23 0.29" rpy="${0*d2r} ${0*d2r} ${135*d2r}"/>
+  <xacro:thruster_macro namespace="${namespace}" parent_link="base_link" thruster_id="8">
+    <origin xyz="${length_1 + length_2 + length_3 + 3*length_joint + 0.715} 0 ${2*radius}" rpy="${0*d2r} ${0*d2r} ${-90*d2r}"/>
   </xacro:thruster_macro>
-  <xacro:thruster_macro namespace="${namespace}" thruster_id="1">
-    <origin xyz="0.48 -0.23 0.29" rpy="${0*d2r} ${0*d2r} ${-135*d2r}"/>
-  <xacro:thruster_macro namespace="${namespace}" thruster_id="0">
-    <origin xyz="-0.890895 0.334385 0.528822" rpy="${0*d2r} ${0*d2r} ${0*d2r}"/>
+  <xacro:thruster_macro namespace="${namespace}" parent_link="base_link" thruster_id="9">
+    <origin xyz="${length_1 + length_2 + length_3 + 3*length_joint + 0.715} 0 0" rpy="${0*d2r} ${0*d2r} ${90*d2r}"/>
   </xacro:thruster_macro>
-  <xacro:thruster_macro namespace="${namespace}" thruster_id="1">
-    <origin xyz="-0.890895 -0.334385 0.528822" rpy="${0*d2r} ${-74.53*d2r} ${53.21*d2r}"/>
+  <xacro:thruster_macro namespace="${namespace}" parent_link="base_link" thruster_id="10">
+    <origin xyz="${length_1 + length_2 + length_3 + 3*length_joint + 0.815} ${radius+0.08} ${radius}" rpy="${0*d2r} ${45*d2r} ${0*d2r}"/>
   </xacro:thruster_macro>
-  <xacro:thruster_macro namespace="${namespace}" thruster_id="2">
-    <origin xyz="0.890895 0.334385 0.528822" rpy="${0*d2r} ${-105.47*d2r} ${53.21*d2r}"/>
+  <xacro:thruster_macro namespace="${namespace}" parent_link="base_link" thruster_id="11">
+    <origin xyz="${length_1 + length_2 + length_3 + 3*length_joint + 0.815} ${-radius-0.08} ${radius}" rpy="${0*d2r} ${-45*d2r} ${0*d2r}"/>
   </xacro:thruster_macro>
-  <xacro:thruster_macro namespace="${namespace}" thruster_id="3">
-    <origin xyz="0.890895 -0.334385 0.528822" rpy="${0*d2r} ${-105.47*d2r} ${-53.21*d2r}"/>
-  </xacro:thruster_macro>
-  <xacro:thruster_macro namespace="${namespace}" thruster_id="4">
-    <origin xyz="-0.412125 0.505415 0.129" rpy="${0*d2r} ${0*d2r} ${45*d2r}"/>
-  </xacro:thruster_macro>
-  <xacro:thruster_macro namespace="${namespace}" thruster_id="5">
-    <origin xyz="-0.412125 -0.505415 0.129" rpy="${0*d2r} ${0*d2r} ${-45*d2r}"/>
-  </xacro:thruster_macro>
-  <xacro:thruster_macro namespace="${namespace}" thruster_id="6">
-    <origin xyz="0.412125 0.505415 0.129" rpy="${0*d2r} ${0*d2r} ${135*d2r}"/>
-  </xacro:thruster_macro>
-  <xacro:thruster_macro namespace="${namespace}" thruster_id="7">
-    <origin xyz="0.412125 -0.505415 0.129" rpy="${0*d2r} ${0*d2r} ${-135*d2r}"/>
-  </xacro:thruster_macro>
-  -->
+-->
+<!-- U-Shape horizontal-->
+<!--
+<xacro:thruster_macro namespace="${namespace}" parent_link="base_link" thruster_id="0">
+  <origin xyz="${length_1/2 + length_joint/2 + 0.707/2*(length_2+length_joint-2*0.12)} ${0.707/2*(length_2+length_joint-2*0.12)} ${radius}" rpy="${0*d2r} ${0*d2r} ${(-45)*d2r}"/>
+</xacro:thruster_macro>
+<xacro:thruster_macro namespace="${namespace}" parent_link="base_link" thruster_id="1">
+  <origin xyz="${length_1/2 + length_joint/2 + 0.707/2*(length_2+length_joint-2*0.12)} ${0.707/2*(length_2+length_joint-2*0.12)} ${-radius}" rpy="${0*d2r} ${0*d2r} ${(135)*d2r}"/>
+</xacro:thruster_macro>
+<xacro:thruster_macro namespace="${namespace}" parent_link="base_link" thruster_id="2">
+  <origin xyz="${length_1/2 + length_joint/2 + 0.707/2*(length_2+length_joint-2*(0.22+radius+0.08))} ${0.707/2*(length_2+length_joint-2*(0.22-radius-0.08))} 0" rpy="${0*d2r} ${45*d2r} ${45*d2r}"/>
+</xacro:thruster_macro>
+<xacro:thruster_macro namespace="${namespace}" parent_link="base_link" thruster_id="3">
+  <origin xyz="${length_1/2 + length_joint/2 + 0.707/2*(length_2+length_joint-2*(0.22-radius-0.08))} ${0.707/2*(length_2+length_joint-2*(0.22+radius+0.08))} 0" rpy="${0*d2r} ${-45*d2r} ${45*d2r}"/>
+</xacro:thruster_macro>
+<xacro:thruster_macro namespace="${namespace}" parent_link="base_link" thruster_id="4">
+  <origin xyz="${length_1/2 + length_joint/2 + 0.707*(length_2+length_joint)} ${0.707*(length_2+length_joint) + (length_3+length_joint)/2-0.042} ${radius}" rpy="${0*d2r} ${0*d2r} ${0*d2r}"/>
+</xacro:thruster_macro>
+<xacro:thruster_macro namespace="${namespace}" parent_link="base_link" thruster_id="5">
+  <origin xyz="${length_1/2 + length_joint/2 + 0.707*(length_2+length_joint)} ${0.707*(length_2+length_joint) + (length_3+length_joint)/2-0.042} ${-radius}" rpy="${0*d2r} ${0*d2r} ${180*d2r}"/>
+</xacro:thruster_macro>
+<xacro:thruster_macro namespace="${namespace}" parent_link="base_link" thruster_id="6">
+  <origin xyz="${length_1/2 + length_joint/2 + 0.707*(length_2+length_joint) +radius+0.08} ${(0.707*(length_2+length_joint) + (length_3+length_joint)/2)+0.058} 0" rpy="${0*d2r} ${-45*d2r} ${90*d2r}"/>
+</xacro:thruster_macro>
+<xacro:thruster_macro namespace="${namespace}" parent_link="base_link" thruster_id="7">
+  <origin xyz="${length_1/2 + length_joint/2 + 0.707*(length_2+length_joint) -radius-0.08} ${(0.707*(length_2+length_joint) + (length_3+length_joint)/2)+0.058} 0" rpy="${0*d2r} ${45*d2r} ${90*d2r}"/>
+</xacro:thruster_macro>
+<xacro:thruster_macro namespace="${namespace}" parent_link="base_link" thruster_id="8">
+  <origin xyz="${length_1/2 + length_joint/2 + 0.707/2*(length_4+length_joint) -0.707*0.12} ${0.707*(length_2+length_joint + 0.12)+(length_3+length_joint)+0.707/2*(length_4+length_joint)} ${radius}" rpy="${0*d2r} ${0*d2r} ${45*d2r}"/>
+</xacro:thruster_macro>
+<xacro:thruster_macro namespace="${namespace}" parent_link="base_link" thruster_id="9">
+  <origin xyz="${length_1/2 + length_joint/2 + 0.707/2*(length_4+length_joint) -0.707*0.12} ${0.707*(length_2+length_joint + 0.12)+(length_3+length_joint)+0.707/2*(length_4+length_joint)} ${-radius}" rpy="${0*d2r} ${0*d2r} ${225*d2r}"/>
+</xacro:thruster_macro>
+<xacro:thruster_macro namespace="${namespace}" parent_link="base_link" thruster_id="10">
+  <origin xyz="${length_1/2 + length_joint/2 + 0.707/2*(length_4+length_joint) +0.707*(-0.22+radius+0.08)} ${0.707*(length_2+length_joint+0.22+radius+0.08)+(length_3+length_joint)+0.707/2*(length_4+length_joint)} 0" rpy="${0*d2r} ${-45*d2r} ${135*d2r}"/>
+</xacro:thruster_macro>
+<xacro:thruster_macro namespace="${namespace}" parent_link="base_link" thruster_id="11">
+  <origin xyz="${length_1/2 + length_joint/2 + 0.707/2*(length_4+length_joint) +0.707*(-0.22-radius-0.08)} ${0.707*(length_2+length_joint+0.22-radius-0.08)+(length_3+length_joint)+0.707/2*(length_4+length_joint)} 0" rpy="${0*d2r} ${45*d2r} ${135*d2r}"/>
+</xacro:thruster_macro>
+-->
+<!-- U-Shape vertical-->
+<!-- -->
+<xacro:thruster_macro namespace="${namespace}" parent_link="base_link" thruster_id="0">
+  <origin xyz="${length_1/2 + length_joint/2 + 0.707/2*(length_2+length_joint-2*0.12+2*radius)} 0 ${-0.707/2*(length_2+length_joint-2*(0.12))+0.707*radius}" rpy="${0*d2r} ${0*d2r} ${-90*d2r}"/>
+</xacro:thruster_macro>
+<xacro:thruster_macro namespace="${namespace}" parent_link="base_link" thruster_id="1">
+  <origin xyz="${length_1/2 + length_joint/2 + 0.707/2*(length_2+length_joint-2*0.12-2*radius)} 0 ${-0.707/2*(length_2+length_joint-2*(0.12))-0.707*radius}" rpy="${0*d2r} ${0*d2r} ${90*d2r}"/>
+</xacro:thruster_macro>
+<xacro:thruster_macro namespace="${namespace}" parent_link="base_link" thruster_id="2">
+  <origin xyz="${length_1/2 + length_joint/2 + 0.707/2*(length_2+length_joint-2*(0.22))} ${radius+0.08} ${-0.707/2*(length_2+length_joint-2*(0.22))}" rpy="${0*d2r} ${90*d2r} ${0*d2r}"/>
+</xacro:thruster_macro>
+<xacro:thruster_macro namespace="${namespace}" parent_link="base_link" thruster_id="3">
+  <origin xyz="${length_1/2 + length_joint/2 + 0.707/2*(length_2+length_joint-2*(0.22))} ${-radius-0.08} ${-0.707/2*(length_2+length_joint-2*(0.22))}" rpy="${0*d2r} ${0*d2r} ${0*d2r}"/>
+</xacro:thruster_macro>
+<xacro:thruster_macro namespace="${namespace}" parent_link="base_link" thruster_id="4">
+  <origin xyz="${length_1/2 + length_joint/2 + 0.707*(length_2+length_joint) +radius} 0 ${-0.707*(length_2+length_joint) - (length_3+length_joint)/2+0.042}" rpy="${0*d2r} ${0*d2r} ${-90*d2r}"/>
+</xacro:thruster_macro>
+<xacro:thruster_macro namespace="${namespace}" parent_link="base_link" thruster_id="5">
+  <origin xyz="${length_1/2 + length_joint/2 + 0.707*(length_2+length_joint) -radius} 0 ${-0.707*(length_2+length_joint) - (length_3+length_joint)/2+0.042}" rpy="${0*d2r} ${0*d2r} ${90*d2r}"/>
+</xacro:thruster_macro>
+<xacro:thruster_macro namespace="${namespace}" parent_link="base_link" thruster_id="6">
+  <origin xyz="${length_1/2 + length_joint/2 + 0.707*(length_2+length_joint)} ${radius+0.08} ${-(0.707*(length_2+length_joint) + (length_3+length_joint)/2)-0.058}" rpy="${0*d2r} ${135*d2r} ${0*d2r}"/>
+</xacro:thruster_macro>
+<xacro:thruster_macro namespace="${namespace}" parent_link="base_link" thruster_id="7">
+  <origin xyz="${length_1/2 + length_joint/2 + 0.707*(length_2+length_joint)} ${-radius-0.08} ${-(0.707*(length_2+length_joint) + (length_3+length_joint)/2)-0.058}" rpy="${0*d2r} ${45*d2r} ${0*d2r}"/>
+</xacro:thruster_macro>
+<xacro:thruster_macro namespace="${namespace}" parent_link="base_link" thruster_id="8">
+  <origin xyz="${length_1/2 + length_joint/2 + 0.707/2*(length_4+length_joint) -0.707*(0.12-radius)} 0 ${-0.707*(length_2+length_joint + 0.12+radius)-(length_3+length_joint)-0.707/2*(length_4+length_joint)}" rpy="${0*d2r} ${0*d2r} ${-90*d2r}"/>
+</xacro:thruster_macro>
+<xacro:thruster_macro namespace="${namespace}" parent_link="base_link" thruster_id="9">
+  <origin xyz="${length_1/2 + length_joint/2 + 0.707/2*(length_4+length_joint) -0.707*(0.12+radius)} 0 ${-0.707*(length_2+length_joint + 0.12-radius)-(length_3+length_joint)-0.707/2*(length_4+length_joint)}" rpy="${0*d2r} ${0*d2r} ${90*d2r}"/>
+</xacro:thruster_macro>
+<xacro:thruster_macro namespace="${namespace}" parent_link="base_link" thruster_id="10">
+  <origin xyz="${length_1/2 + length_joint/2 + 0.707/2*(length_4+length_joint) +0.707*(-0.22)} ${radius+0.08} ${-0.707*(length_2+length_joint+0.22)-(length_3+length_joint)-0.707/2*(length_4+length_joint)}" rpy="${0*d2r} ${180*d2r} ${0*d2r}"/>
+</xacro:thruster_macro>
+<xacro:thruster_macro namespace="${namespace}" parent_link="base_link" thruster_id="11">
+  <origin xyz="${length_1/2 + length_joint/2 + 0.707/2*(length_4+length_joint) +0.707*(-0.22)} ${-radius-0.08} ${-0.707*(length_2+length_joint+0.22)-(length_3+length_joint)-0.707/2*(length_4+length_joint)}" rpy="${0*d2r} ${90*d2r} ${0*d2r}"/>
+</xacro:thruster_macro>
 </robot>
